File: resources/kicad/pro_micro_shield/pro_micro_shield.sch (KiCad schematic (older format))
At the start: 19 parts, among them U0 ProMicro

Commit message: shield pcb revision 2
Parts:
- removed JGND0, JGND1, JPIN0, JPIN1, JVCC0, JVCC1: Conn_01x01_Female, Connector_Wire:SolderWirePad_1x01_Drill1mm, symbol Connector:Conn_01x01_Female
- removed JL0, JL1, JL2: Conn_01x02_Female, Connector_Wire:SolderWirePad_1x02_P3.81mm_Drill1mm, symbol Connector:Conn_01x02_Female
- added JEX0, JEX1: Conn_01x03_Female, Connector_Wire:SolderWirePad_1x03_P3.175mm_Drill1mm, symbol Connector:Conn_01x03_Female
Connections:
- net GND: now also JEX0.2 (Pin_2), JEX1.2 (Pin_2)
- net VCC: now also JEX0.1 (Pin_1), JEX1.1 (Pin_1)
- net at JRGB0.2 (Pin_2), U0.6 (SDA): now also JRGB1.2 (Pin_2)
- net at U0.7 (D4): now also JEX1.3 (Pin_3); no longer JRGB1.2 (Pin_2)
- net at U0.8 (C6): now also JEX0.3 (Pin_3)
- no-connect marks 11 -> 13
Changed lines of the file:
@@
-	1    0    0    -1
-$EndComp
-$Comp
-L Connector:Conn_01x02_Female JL0
-U 1 1 5E63EBB8
-P 5850 4950
-F 0 "JL0" H 5878 4926 50  0000 L CNN
-F 1 "Conn_01x02_Female" H 5878 4835 50  0000 L CNN
-F 2 "Connector_Wire:SolderWirePad_1x02_P3.81mm_Drill1mm" H 5850 4950 50  0001 C CNN
-F 3 "~" H 5850 4950 50  0001 C CNN
-	1    5850 4950
-	1    0    0    -1
-$EndComp
-$Comp
-L Connector:Conn_01x02_Female JL1
-U 1 1 5E63F977
-P 5850 5200
-F 0 "JL1" H 5878 5176 50  0000 L CNN
-F 1 "Conn_01x02_Female" H 5878 5085 50  0000 L CNN
-F 2 "Connector_Wire:SolderWirePad_1x02_P3.81mm_Drill1mm" H 5850 5200 50  0001 C CNN
-F 3 "~" H 5850 5200 50  0001 C CNN
-	1    5850 5200
-	1    0    0    -1
-$EndComp
-$Comp
-L Connector:Conn_01x02_Female JL2
-U 1 1 5E64015B
-P 5850 5450
-F 0 "JL2" H 5878 5426 50  0000 L CNN
-F 1 "Conn_01x02_Female" H 5878 5335 50  0000 L CNN
-F 2 "Connector_Wire:SolderWirePad_1x02_P3.81mm_Drill1mm" H 5850 5450 50  0001 C CNN
-F 3 "~" H 5850 5450 50  0001 C CNN
-	1    5850 5450
-	1    0    0    -1
-$EndComp
-$Comp
-L Connector:Conn_01x02_Female JSPEAKER0
-U 1 1 5E640A6C
-P 5850 5700
-F 0 "JSPEAKER0" H 5878 5676 50  0000 L CNN
-F 1 "Conn_01x02_Female" H 5878 5585 50  0000 L CNN
-F 2 "Connector_Wire:SolderWirePad_1x02_P3.81mm_Drill1mm" H 5850 5700 50  0001 C CNN
-F 3 "~" H 5850 5700 50  0001 C CNN
-	1    5850 5700
 	1    0    0    -1
 $EndComp
@@
 Text GLabel 5650 4650 0    50   Input ~ 0
 VCC
-Text GLabel 5650 4950 0    50   Input ~ 0
-GND
-Text GLabel 5650 5200 0    50   Input ~ 0
-GND
-Text GLabel 5650 5450 0    50   Input ~ 0
-GND
 Text GLabel 5650 5700 0    50   Input ~ 0
 GND
@@
 	3000 3500 3300 3500
 Wire Wire Line
-	5650 5050 5300 5050
-Wire Wire Line
 	3200 4950 3200 3600
 Wire Wire Line
 	3200 3600 3300 3600
 Wire Wire Line
-	5650 5300 5200 5300
-Wire Wire Line
 	3150 5200 3150 3700
 Wire Wire Line
 	3150 3700 3300 3700
-Wire Wire Line
-	5650 5550 3100 5550
 Wire Wire Line
 	3100 3800 3300 3800
@@
 	5650 4200 5300 4200
 Wire Wire Line
-	5300 4200 5300 4950
-Wire Wire Line
 	5300 4950 3200 4950
-Wire Wire Line
-	5650 4550 5200 4550
-Wire Wire Line
-	5200 4550 5200 5200
-Wire Wire Line
-	5200 5200 3150 5200
-Text GLabel 7000 3000 0    50   Input ~ 0
-GND
-Text GLabel 7000 3100 0    50   Input ~ 0
-GND
-Text GLabel 7000 3350 0    50   Input ~ 0
-VCC
-Text GLabel 7000 3450 0    50   Input ~ 0
-VCC
-Wire Wire Line
-	7000 3700 6800 3700
-Wire Wire Line
-	6800 4750 3300 4750
-Wire Wire Line
-	3300 4750 3300 4200
-Wire Wire Line
-	7000 3800 6850 3800
-Wire Wire Line
-	6850 3800 6850 4800
-Wire Wire Line
-	6850 4800 4800 4800
-Wire Wire Line
-	4800 4800 4800 4200
-Wire Wire Line
-	4800 4200 4700 4200
 NoConn ~ 4700 3100
 NoConn ~ 4700 3300
@@
 NoConn ~ 3300 3200
 Wire Wire Line
-	5300 5050 5300 4950
-Connection ~ 5300 4950
-Wire Wire Line
-	5200 5300 5200 5200
-Connection ~ 5200 5200
-Wire Wire Line
 	3100 3800 3100 5550
 Wire Wire Line
 	3000 3500 3000 5800
-$Comp
-L Connector:Conn_01x01_Female JPIN0
-U 1 1 5E66D93E
-P 7200 3700
-F 0 "JPIN0" H 7228 3726 50  0000 L CNN
-F 1 "Conn_01x01_Female" H 7228 3635 50  0000 L CNN
-F 2 "Connector_Wire:SolderWirePad_1x01_Drill1mm" H 7200 3700 50  0001 C CNN
-F 3 "~" H 7200 3700 50  0001 C CNN
-	1    7200 3700
-	1    0    0    -1
-$EndComp
-Wire Wire Line
-	6800 3700 6800 4750
-$Comp
-L Connector:Conn_01x01_Female JPIN1
-U 1 1 5E66E582
-P 7200 3800
-F 0 "JPIN1" H 7228 3826 50  0000 L CNN
-F 1 "Conn_01x01_Female" H 7228 3735 50  0000 L CNN
-F 2 "Connector_Wire:SolderWirePad_1x01_Drill1mm" H 7200 3800 50  0001 C CNN
-F 3 "~" H 7200 3800 50  0001 C CNN
-	1    7200 3800
-	1    0    0    -1
-$EndComp
 $Comp
 L Mechanical:MountingHole H0
@@
 Text GLabel 7250 4050 0    50   Input ~ 0
 GND
+Wire Wire Line
+	5300 4200 5300 4550
 $Comp
-L Connector:Conn_01x01_Female JGND0
-U 1 1 5E666EF2
-P 7200 3000
-F 0 "JGND0" H 7228 3026 50  0000 L CNN
-F 1 "Conn_01x01_Female" H 7228 2935 50  0000 L CNN
-F 2 "Connector_Wire:SolderWirePad_1x01_Drill1mm" H 7200 3000 50  0001 C CNN
-F 3 "~" H 7200 3000 50  0001 C CNN
-	1    7200 3000
+L Connector:Conn_01x02_Female JSPEAKER0
+U 1 1 5E640A6C
+P 5850 5700
+F 0 "JSPEAKER0" H 5878 5676 50  0000 L CNN
+F 1 "Conn_01x02_Female" H 5878 5585 50  0000 L CNN
+F 2 "Connector_Wire:SolderWirePad_1x02_P3.81mm_Drill1mm" H 5850 5700 50  0001 C CNN
+F 3 "~" H 5850 5700 50  0001 C CNN
+	1    5850 5700
 	1    0    0    -1
 $EndComp
+Wire Wire Line
+	5650 4550 5300 4550
+Connection ~ 5300 4550
+Wire Wire Line
+	5300 4550 5300 4950
 $Comp
-L Connector:Conn_01x01_Female JGND1
-U 1 1 5E667A92
-P 7200 3100
-F 0 "JGND1" H 7228 3126 50  0000 L CNN
-F 1 "Conn_01x01_Female" H 7228 3035 50  0000 L CNN
-F 2 "Connector_Wire:SolderWirePad_1x01_Drill1mm" H 7200 3100 50  0001 C CNN
-F 3 "~" H 7200 3100 50  0001 C CNN
-	1    7200 3100
+L Connector:Conn_01x03_Female JEX0
+U 1 1 5F92E86A
+P 5850 5450
+F 0 "JEX0" H 5878 5476 50  0000 L CNN
+F 1 "Conn_01x03_Female" H 5878 5385 50  0000 L CNN
+F 2 "Connector_Wire:SolderWirePad_1x03_P3.175mm_Drill1mm" H 5850 5450 50  0001 C CNN
+F 3 "~" H 5850 5450 50  0001 C CNN
+	1    5850 5450
 	1    0    0    -1
 $EndComp
+Text GLabel 5650 5350 0    50   Input ~ 0
+VCC
+Text GLabel 5650 5450 0    50   Input ~ 0
+GND
 $Comp
-L Connector:Conn_01x01_Female JVCC0
-U 1 1 5E6684FC
-P 7200 3350
-F 0 "JVCC0" H 7228 3376 50  0000 L CNN
-F 1 "Conn_01x01_Female" H 7228 3285 50  0000 L CNN
-F 2 "Connector_Wire:SolderWirePad_1x01_Drill1mm" H 7200 3350 50  0001 C CNN
-F 3 "~" H 7200 3350 50  0001 C CNN
-	1    7200 3350
+L Connector:Conn_01x03_Female JEX1
+U 1 1 5F930EE7
+P 5850 5100
+F 0 "JEX1" H 5878 5126 50  0000 L CNN
+F 1 "Conn_01x03_Female" H 5878 5035 50  0000 L CNN
+F 2 "Connector_Wire:SolderWirePad_1x03_P3.175mm_Drill1mm" H 5850 5100 50  0001 C CNN
+F 3 "~" H 5850 5100 50  0001 C CNN
+	1    5850 5100
 	1    0    0    -1
 $EndComp
-$Comp
-L Connector:Conn_01x01_Female JVCC1
-U 1 1 5E6689E2
-P 7200 3450
-F 0 "JVCC1" H 7228 3476 50  0000 L CNN
-F 1 "Conn_01x01_Female" H 7228 3385 50  0000 L CNN
-F 2 "Connector_Wire:SolderWirePad_1x01_Drill1mm" H 7200 3450 50  0001 C CNN
-F 3 "~" H 7200 3450 50  0001 C CNN
-	1    7200 3450
-	1    0    0    -1
-$EndComp
+Text GLabel 5650 5000 0    50   Input ~ 0
+VCC
+Text GLabel 5650 5100 0    50   Input ~ 0
+GND
+Wire Wire Line
+	5650 5200 3150 5200
+Wire Wire Line
+	3100 5550 5650 5550
+NoConn ~ 4700 4200
+NoConn ~ 3300 4200
 $EndSCHEMATC

Commit message: update gerber for shield
Parts:
- renumbered JEX0 to JBTN0, JEX1 to JEX0
Connections:
- net at U0.12 (B5): now also JBTN0.3 (Pin_3)
- net at U0.8 (C6): no longer JBTN0.3 (Pin_3)
Changed lines of the file:
@@
 	3150 3700 3300 3700
-Wire Wire Line
-	3100 3800 3300 3800
 Wire Wire Line
 	5650 3250 5000 3250
@@
 NoConn ~ 3300 3100
 NoConn ~ 3300 3200
-Wire Wire Line
-	3100 3800 3100 5550
 Wire Wire Line
 	3000 3500 3000 5800
@@
 	5300 4550 5300 4950
 $Comp
-L Connector:Conn_01x03_Female JEX0
+L Connector:Conn_01x03_Female JBTN0
 U 1 1 5F92E86A
 P 5850 5450
-F 0 "JEX0" H 5878 5476 50  0000 L CNN
+F 0 "JBTN0" H 5878 5476 50  0000 L CNN
 F 1 "Conn_01x03_Female" H 5878 5385 50  0000 L CNN
 F 2 "Connector_Wire:SolderWirePad_1x03_P3.175mm_Drill1mm" H 5850 5450 50  0001 C CNN
@@
 GND
 $Comp
-L Connector:Conn_01x03_Female JEX1
+L Connector:Conn_01x03_Female JEX0
 U 1 1 5F930EE7
 P 5850 5100
-F 0 "JEX1" H 5878 5126 50  0000 L CNN
+F 0 "JEX0" H 5878 5126 50  0000 L CNN
 F 1 "Conn_01x03_Female" H 5878 5035 50  0000 L CNN
 F 2 "Connector_Wire:SolderWirePad_1x03_P3.175mm_Drill1mm" H 5850 5100 50  0001 C CNN
@@
 	3100 5550 5650 5550
 NoConn ~ 4700 4200
-NoConn ~ 3300 4200
+Wire Wire Line
+	3100 5550 3100 4200
+Wire Wire Line
+	3100 4200 3300 4200
+NoConn ~ 3300 3800
 $EndSCHEMATC

Commit message: cleanup resources and shield gerber files
Parts:
- removed JBTN0: Conn_01x03_Female, Connector_Wire:SolderWirePad_1x03_P3.175mm_Drill1mm, symbol Connector:Conn_01x03_Female
- added H2: MountingHole, MountingHole:MountingHole_2.2mm_M2, symbol Mechanical:MountingHole
- added JBUTTON0: Conn_01x02_Female, Connector_Wire:SolderWirePad_1x02_P3.81mm_Drill1mm, symbol Connector:Conn_01x02_Female
- added R0: R_US, Resistor_THT:R_Axial_DIN0207_L6.3mm_D2.5mm_P7.62mm_Horizontal, symbol Device:R_US
Connections:
- net GND: now also R0.2
- net VCC: now also JBUTTON0.1 (Pin_1)
- net at U0.12 (B5): now also JBUTTON0.2 (Pin_2), R0.1
Changed lines of the file:
@@
 Wire Wire Line
 	5300 4550 5300 4950
-$Comp
-L Connector:Conn_01x03_Female JBTN0
-U 1 1 5F92E86A
-P 5850 5450
-F 0 "JBTN0" H 5878 5476 50  0000 L CNN
-F 1 "Conn_01x03_Female" H 5878 5385 50  0000 L CNN
-F 2 "Connector_Wire:SolderWirePad_1x03_P3.175mm_Drill1mm" H 5850 5450 50  0001 C CNN
-F 3 "~" H 5850 5450 50  0001 C CNN
-	1    5850 5450
-	1    0    0    -1
-$EndComp
-Text GLabel 5650 5350 0    50   Input ~ 0
+Text GLabel 5650 5450 0    50   Input ~ 0
 VCC
-Text GLabel 5650 5450 0    50   Input ~ 0
+Text GLabel 4950 5450 0    50   Input ~ 0
 GND
 $Comp
@@
 	5650 5200 3150 5200
 Wire Wire Line
-	3100 5550 5650 5550
+	3100 5550 5250 5550
 NoConn ~ 4700 4200
 Wire Wire Line
@@
 	3100 4200 3300 4200
 NoConn ~ 3300 3800
+$Comp
+L Mechanical:MountingHole H2
+U 1 1 5FD3A4F1
+P 7350 5050
+F 0 "H2" H 7450 5096 50  0000 L CNN
+F 1 "MountingHole" H 7450 5005 50  0000 L CNN
+F 2 "MountingHole:MountingHole_2.2mm_M2" H 7350 5050 50  0001 C CNN
+F 3 "~" H 7350 5050 50  0001 C CNN
+	1    7350 5050
+	1    0    0    -1
+$EndComp
+$Comp
+L Device:R_US R0
+U 1 1 5FD3B002
+P 5100 5450
+F 0 "R0" V 4895 5450 50  0000 C CNN
+F 1 "R_US" V 4986 5450 50  0000 C CNN
+F 2 "Resistor_THT:R_Axial_DIN0207_L6.3mm_D2.5mm_P7.62mm_Horizontal" V 5140 5440 50  0001 C CNN
+F 3 "~" H 5100 5450 50  0001 C CNN
+	1    5100 5450
+	0    1    1    0
+$EndComp
+$Comp
+L Connector:Conn_01x02_Female JBUTTON0
+U 1 1 5FD41B09
+P 5850 5450
+F 0 "JBUTTON0" H 5878 5426 50  0000 L CNN
+F 1 "Conn_01x02_Female" H 5878 5335 50  0000 L CNN
+F 2 "Connector_Wire:SolderWirePad_1x02_P3.81mm_Drill1mm" H 5850 5450 50  0001 C CNN
+F 3 "~" H 5850 5450 50  0001 C CNN
+	1    5850 5450
+	1    0    0    -1
+$EndComp
+Wire Wire Line
+	5250 5450 5250 5550
+Connection ~ 5250 5550
+Wire Wire Line
+	5250 5550 5650 5550
 $EndSCHEMATC

Commit message: use standard 2.54mm header pins in arduino shield
Parts:
- JBUTTON0, JLASER0, JSPEAKER0: footprint Connector_Wire:SolderWirePad_1x02_P3.81mm_Drill1mm -> Connector_PinHeader_2.54mm:PinHeader_1x02_P2.54mm_Vertical
- JEX0, JRGB0, JRGB1, JS0, JS1, JS2: footprint Connector_Wire:SolderWirePad_1x03_P3.175mm_Drill1mm -> Connector_PinHeader_2.54mm:PinHeader_1x03_P2.54mm_Vertical
Changed lines of the file:
@@
 F 0 "JS0" H 5878 3176 50  0000 L CNN
 F 1 "Conn_01x03_Female" H 5878 3085 50  0000 L CNN
-F 2 "Connector_Wire:SolderWirePad_1x03_P3.175mm_Drill1mm" H 5850 3150 50  0001 C CNN
+F 2 "Connector_PinHeader_2.54mm:PinHeader_1x03_P2.54mm_Vertical" H 5850 3150 50  0001 C CNN
 F 3 "~" H 5850 3150 50  0001 C CNN
 	1    5850 3150
@@
 F 0 "JS1" H 5878 3526 50  0000 L CNN
 F 1 "Conn_01x03_Female" H 5878 3435 50  0000 L CNN
-F 2 "Connector_Wire:SolderWirePad_1x03_P3.175mm_Drill1mm" H 5850 3500 50  0001 C CNN
+F 2 "Connector_PinHeader_2.54mm:PinHeader_1x03_P2.54mm_Vertical" H 5850 3500 50  0001 C CNN
 F 3 "~" H 5850 3500 50  0001 C CNN
 	1    5850 3500
@@
 F 0 "JS2" H 5878 3876 50  0000 L CNN
 F 1 "Conn_01x03_Female" H 5878 3785 50  0000 L CNN
-F 2 "Connector_Wire:SolderWirePad_1x03_P3.175mm_Drill1mm" H 5850 3850 50  0001 C CNN
+F 2 "Connector_PinHeader_2.54mm:PinHeader_1x03_P2.54mm_Vertical" H 5850 3850 50  0001 C CNN
 F 3 "~" H 5850 3850 50  0001 C CNN
 	1    5850 3850
@@
 F 0 "JRGB0" H 5878 4226 50  0000 L CNN
 F 1 "Conn_01x03_Female" H 5878 4135 50  0000 L CNN
-F 2 "Connector_Wire:SolderWirePad_1x03_P3.175mm_Drill1mm" H 5850 4200 50  0001 C CNN
+F 2 "Connector_PinHeader_2.54mm:PinHeader_1x03_P2.54mm_Vertical" H 5850 4200 50  0001 C CNN
 F 3 "~" H 5850 4200 50  0001 C CNN
 	1    5850 4200
@@
 F 0 "JRGB1" H 5878 4576 50  0000 L CNN
 F 1 "Conn_01x03_Female" H 5878 4485 50  0000 L CNN
-F 2 "Connector_Wire:SolderWirePad_1x03_P3.175mm_Drill1mm" H 5850 4550 50  0001 C CNN
+F 2 "Connector_PinHeader_2.54mm:PinHeader_1x03_P2.54mm_Vertical" H 5850 4550 50  0001 C CNN
 F 3 "~" H 5850 4550 50  0001 C CNN
 	1    5850 4550
@@
 F 0 "JLASER0" H 7478 4026 50  0000 L CNN
 F 1 "Conn_01x02_Female" H 7478 3935 50  0000 L CNN
-F 2 "Connector_Wire:SolderWirePad_1x02_P3.81mm_Drill1mm" H 7450 4050 50  0001 C CNN
+F 2 "Connector_PinHeader_2.54mm:PinHeader_1x02_P2.54mm_Vertical" H 7450 4050 50  0001 C CNN
 F 3 "~" H 7450 4050 50  0001 C CNN
 	1    7450 4050
@@
 F 0 "JSPEAKER0" H 5878 5676 50  0000 L CNN
 F 1 "Conn_01x02_Female" H 5878 5585 50  0000 L CNN
-F 2 "Connector_Wire:SolderWirePad_1x02_P3.81mm_Drill1mm" H 5850 5700 50  0001 C CNN
+F 2 "Connector_PinHeader_2.54mm:PinHeader_1x02_P2.54mm_Vertical" H 5850 5700 50  0001 C CNN
 F 3 "~" H 5850 5700 50  0001 C CNN
 	1    5850 5700
@@
 F 0 "JEX0" H 5878 5126 50  0000 L CNN
 F 1 "Conn_01x03_Female" H 5878 5035 50  0000 L CNN
-F 2 "Connector_Wire:SolderWirePad_1x03_P3.175mm_Drill1mm" H 5850 5100 50  0001 C CNN
+F 2 "Connector_PinHeader_2.54mm:PinHeader_1x03_P2.54mm_Vertical" H 5850 5100 50  0001 C CNN
 F 3 "~" H 5850 5100 50  0001 C CNN
 	1    5850 5100
@@
 F 0 "JBUTTON0" H 5878 5426 50  0000 L CNN
 F 1 "Conn_01x02_Female" H 5878 5335 50  0000 L CNN
-F 2 "Connector_Wire:SolderWirePad_1x02_P3.81mm_Drill1mm" H 5850 5450 50  0001 C CNN
+F 2 "Connector_PinHeader_2.54mm:PinHeader_1x02_P2.54mm_Vertical" H 5850 5450 50  0001 C CNN
 F 3 "~" H 5850 5450 50  0001 C CNN
 	1    5850 5450
