File: resources/kicad/pro_micro_shield/pro_micro_shield.kicad_pcb (KiCad board)
At the start: 2 copper layers, 34.5 x 45.8 mm, 19 parts, among them U0 ProMicro

Commit message: shield pcb revision 2
Parts:
- removed JGND0, JGND1, JPIN0, JPIN1, JVCC0, JVCC1: Conn_01x01_Female, Connector_Wire:SolderWirePad_1x01_Drill1mm
- removed JL0, JL1, JL2: Conn_01x02_Female, Connector_Wire:SolderWirePad_1x02_P3.81mm_Drill1mm
- added JEX0: Conn_01x03_Female, Connector_Wire:SolderWirePad_1x03_P3.175mm_Drill1mm, F.Cu at (160.0, 90.5)
- added JEX1: Conn_01x03_Female, Connector_Wire:SolderWirePad_1x03_P3.175mm_Drill1mm, F.Cu at (160.0, 80.0)
- moved JRGB0 34.9 mm to (165.5, 113.5), turned to 0 degrees
- moved JRGB1 28.2 mm to (177.0, 113.5), turned to 0 degrees
- moved JSPEAKER0 9.19 mm to (167.2, 107.2)
- moved JLASER0 7.50 mm to (177.8, 107.2)
- moved JS0 4.50 mm to (189.0, 84.2)
- moved JS1 4.50 mm to (189.0, 94.8)
- moved JS2 4.50 mm to (189.0, 105.2)
Connections:
- JRGB0 pad 2: Net-(JL0-Pad2) -> Net-(JRGB0-Pad2)
- JRGB1 pad 2: Net-(JL1-Pad2) -> Net-(JRGB0-Pad2)
- U0 pad 6: Net-(JL0-Pad2) -> Net-(JRGB0-Pad2)
- U0 pad 7: Net-(JL1-Pad2) -> Net-(JEX1-Pad3)
Routing:
- net Net-(JL1-Pad2): track 46.8 -> 0.00 mm
- net Net-(JRGB0-Pad2): track 0.00 -> 44.0 mm
- net Net-(JL0-Pad2): track 42.3 -> 0.00 mm
- net Net-(JEX0-Pad3): track 42.2 -> 9.38 mm
- net Net-(U0-Pad12): track 12.9 -> 0.00 mm
- net Net-(JSPEAKER0-Pad2): track 34.3 -> 25.8 mm
- net Net-(U0-Pad13): track 7.71 -> 0.00 mm
- net Net-(JEX1-Pad3): track 0.00 -> 7.68 mm
- net Net-(JS1-Pad3): track 40.7 -> 37.5 mm
- net Net-(JS0-Pad3): track 51.4 -> 48.4 mm
- net Net-(JS2-Pad3): track 30.0 -> 27.0 mm
- added copper zone on F.Cu, net GND
- added copper zone on B.Cu, net VCC
- removed copper zone on B.Cu, net GND
- removed copper zone on F.Cu, net VCC
Other:
- board text added: "EXTRA 1"
- board text added: "EXTRA 2"
- board text added: "Mini4wdChrono Shield Rev.2"
- board text removed: "D10"
- board text removed: "D9"
- board text removed: "LED 1"
- board text removed: "LED 2"
- board text removed: "LED 3"
- board text removed: "Mini4wdChrono Shield Rev.1"
- board text removed: "extra connections"

Commit message: update gerber for shield
Parts:
- renumbered JEX0 to JBTN0, JEX1 to JEX0
Connections:
- JBTN0 pad 3: Net-(JEX0-Pad3) (its old number) -> Net-(JBTN0-Pad3)
- U0 pad 12: Net-(U0-Pad12) -> Net-(JBTN0-Pad3)
- U0 pad 8: Net-(JEX0-Pad3) (its old number) -> Net-(U0-Pad8)
Routing:
- net Net-(JEX0-Pad3) (its old number): track 9.38 -> 0.00 mm
- net Net-(JBTN0-Pad3): track 0.00 -> 8.59 mm
Other:
- board text added: "D9"
- board text added: "EXTRA"
- board text added: "START BUTTON"
- board text removed: "D5"
- board text removed: "EXTRA 1"
- board text removed: "EXTRA 2"
Changed lines of the file:
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@@
   (net 17 "Net-(JSPEAKER0-Pad2)")
   (net 18 "Net-(JEX0-Pad3)")
-  (net 19 "Net-(JEX1-Pad3)")
-  (net 20 "Net-(JRGB0-Pad2)")
-  (net 21 "Net-(U0-Pad13)")
-  (net 22 "Net-(U0-Pad12)")
+  (net 19 "Net-(JRGB0-Pad2)")
+  (net 20 "Net-(U0-Pad13)")
+  (net 21 "Net-(JBTN0-Pad3)")
+  (net 22 "Net-(U0-Pad8)")
   (net_class Default "This is the default net class."
     (clearance 0.2)
@@
     (uvia_drill 0.1)
     (add_net GND)
+    (add_net "Net-(JBTN0-Pad3)")
     (add_net "Net-(JEX0-Pad3)")
-    (add_net "Net-(JEX1-Pad3)")
     (add_net "Net-(JRGB0-Pad2)")
     (add_net "Net-(JS0-Pad3)")
@@
     (add_net "Net-(JSPEAKER0-Pad2)")
     (add_net "Net-(U0-Pad1)")
-    (add_net "Net-(U0-Pad12)")
     (add_net "Net-(U0-Pad13)")
     (add_net "Net-(U0-Pad14)")
@@
     (add_net "Net-(U0-Pad22)")
     (add_net "Net-(U0-Pad24)")
+    (add_net "Net-(U0-Pad8)")
     (add_net VCC)
   )
@@
     (tags connector)
     (attr virtual)
-    (fp_text reference JEX1 (at 3.175 -3.81 90) (layer F.SilkS) hide
+    (fp_text reference JEX0 (at 3.175 -3.81 90) (layer F.SilkS) hide
       (effects (font (size 1 1) (thickness 0.15)))
     )
@@
     )
     (pad 3 thru_hole circle (at 6.35 0 270) (size 2.49936 2.49936) (drill 1.00076) (layers *.Cu *.Mask)
-      (net 19 "Net-(JEX1-Pad3)"))
+      (net 18 "Net-(JEX0-Pad3)"))
     (pad 2 thru_hole circle (at 3.175 0 270) (size 2.49936 2.49936) (drill 1.00076) (layers *.Cu *.Mask)
       (net 1 GND))
@@
     (tags connector)
     (attr virtual)
-    (fp_text reference JEX0 (at 3.175 -3.81 90) (layer F.SilkS) hide
+    (fp_text reference JBTN0 (at 3.175 -3.81 90) (layer F.SilkS) hide
       (effects (font (size 1 1) (thickness 0.15)))
     )
@@
     )
     (pad 3 thru_hole circle (at 6.35 0 270) (size 2.49936 2.49936) (drill 1.00076) (layers *.Cu *.Mask)
-      (net 18 "Net-(JEX0-Pad3)"))
+      (net 21 "Net-(JBTN0-Pad3)"))
     (pad 2 thru_hole circle (at 3.175 0 270) (size 2.49936 2.49936) (drill 1.00076) (layers *.Cu *.Mask)
       (net 1 GND))
@@
       (net 6 "Net-(U0-Pad24)"))
     (pad 12 thru_hole circle (at 13.97 7.62 270) (size 1.7526 1.7526) (drill 1.0922) (layers *.Cu *.SilkS *.Mask)
-      (net 22 "Net-(U0-Pad12)"))
+      (net 21 "Net-(JBTN0-Pad3)"))
     (pad 23 thru_hole circle (at -11.43 -7.62 270) (size 1.7526 1.7526) (drill 1.0922) (layers *.Cu *.SilkS *.Mask)
       (net 1 GND))
@@
       (net 14 "Net-(U0-Pad14)"))
     (pad 13 thru_hole circle (at 13.97 -7.62 270) (size 1.7526 1.7526) (drill 1.0922) (layers *.Cu *.SilkS *.Mask)
-      (net 21 "Net-(U0-Pad13)"))
+      (net 20 "Net-(U0-Pad13)"))
     (pad 11 thru_hole circle (at 11.43 7.62 270) (size 1.7526 1.7526) (drill 1.0922) (layers *.Cu *.SilkS *.Mask)
       (net 5 "Net-(JS2-Pad3)"))
@@
       (net 3 "Net-(JS0-Pad3)"))
     (pad 8 thru_hole circle (at 3.81 7.62 270) (size 1.7526 1.7526) (drill 1.0922) (layers *.Cu *.SilkS *.Mask)
+      (net 22 "Net-(U0-Pad8)"))
+    (pad 7 thru_hole circle (at 1.27 7.62 270) (size 1.7526 1.7526) (drill 1.0922) (layers *.Cu *.SilkS *.Mask)
       (net 18 "Net-(JEX0-Pad3)"))
-    (pad 7 thru_hole circle (at 1.27 7.62 270) (size 1.7526 1.7526) (drill 1.0922) (layers *.Cu *.SilkS *.Mask)
-      (net 19 "Net-(JEX1-Pad3)"))
     (pad 6 thru_hole circle (at -1.27 7.62 270) (size 1.7526 1.7526) (drill 1.0922) (layers *.Cu *.SilkS *.Mask)
-      (net 20 "Net-(JRGB0-Pad2)"))
+      (net 19 "Net-(JRGB0-Pad2)"))
     (pad 5 thru_hole circle (at -3.81 7.62 270) (size 1.7526 1.7526) (drill 1.0922) (layers *.Cu *.SilkS *.Mask)
       (net 17 "Net-(JSPEAKER0-Pad2)"))
@@
       (net 2 VCC))
     (pad 2 thru_hole circle (at 3.175 0) (size 2.49936 2.49936) (drill 1.00076) (layers *.Cu *.Mask)
-      (net 20 "Net-(JRGB0-Pad2)"))
+      (net 19 "Net-(JRGB0-Pad2)"))
     (pad 1 thru_hole rect (at 0 0) (size 2.49936 2.49936) (drill 1.00076) (layers *.Cu *.Mask)
       (net 1 GND))
@@
       (net 2 VCC))
     (pad 2 thru_hole circle (at 3.175 0) (size 2.49936 2.49936) (drill 1.00076) (layers *.Cu *.Mask)
-      (net 20 "Net-(JRGB0-Pad2)"))
+      (net 19 "Net-(JRGB0-Pad2)"))
     (pad 1 thru_hole rect (at 0 0) (size 2.49936 2.49936) (drill 1.00076) (layers *.Cu *.Mask)
       (net 1 GND))
@@
     (effects (font (size 1 1) (thickness 0.15)))
   )
-  (gr_text "EXTRA 2" (at 163.5 83 270) (layer F.SilkS)
-    (effects (font (size 1 1) (thickness 0.15)))
-  )
-  (gr_text D5 (at 162 86.5 270) (layer F.SilkS)
+  (gr_text EXTRA (at 163.5 83 270) (layer F.SilkS)
+    (effects (font (size 1 1) (thickness 0.15)))
+  )
+  (gr_text D4 (at 162 86.5 270) (layer F.SilkS)
     (effects (font (size 1 1) (thickness 0.15)))
   )
@@
     (effects (font (size 1 1) (thickness 0.15)))
   )
-  (gr_text D4 (at 162 97 270) (layer F.SilkS)
+  (gr_text D9 (at 162 97 270) (layer F.SilkS)
     (effects (font (size 1 1) (thickness 0.15)))
   )
@@
     (effects (font (size 1 1) (thickness 0.15)))
   )
-  (gr_text "EXTRA 1" (at 163.5 93.5 270) (layer F.SilkS)
+  (gr_text "START BUTTON" (at 163.5 93.5 270) (layer F.SilkS)
     (effects (font (size 1 1) (thickness 0.15)))
   )
@@
   (segment (start 171.06 87.37) (end 166.88 83.19) (width 0.25) (layer B.Cu) (net 17))
   (segment (start 171.06 107.25) (end 171.06 87.37) (width 0.25) (layer B.Cu) (net 17))
-  (segment (start 160.84 96.85) (end 160 96.85) (width 0.25) (layer F.Cu) (net 18))
-  (segment (start 166.88 90.81) (end 160.84 96.85) (width 0.25) (layer F.Cu) (net 18))
-  (segment (start 161.92 88.27) (end 160 86.35) (width 0.25) (layer F.Cu) (net 19))
-  (segment (start 166.88 88.27) (end 161.92 88.27) (width 0.25) (layer F.Cu) (net 19))
-  (segment (start 168.675 113.5) (end 164.25 109.075) (width 0.25) (layer B.Cu) (net 20))
-  (segment (start 168.675 113.5) (end 170.925 111.25) (width 0.25) (layer B.Cu) (net 20))
-  (segment (start 177.925 111.25) (end 180.175 113.5) (width 0.25) (layer B.Cu) (net 20))
-  (segment (start 170.925 111.25) (end 177.925 111.25) (width 0.25) (layer B.Cu) (net 20))
-  (segment (start 164.25 88.36) (end 166.88 85.73) (width 0.25) (layer B.Cu) (net 20))
-  (segment (start 164.25 109) (end 164.25 88.36) (width 0.25) (layer B.Cu) (net 20))
+  (segment (start 161.92 88.27) (end 166.88 88.27) (width 0.25) (layer F.Cu) (net 18))
+  (segment (start 160 86.35) (end 161.92 88.27) (width 0.25) (layer F.Cu) (net 18))
+  (segment (start 168.675 113.5) (end 164.25 109.075) (width 0.25) (layer B.Cu) (net 19))
+  (segment (start 168.675 113.5) (end 170.925 111.25) (width 0.25) (layer B.Cu) (net 19))
+  (segment (start 177.925 111.25) (end 180.175 113.5) (width 0.25) (layer B.Cu) (net 19))
+  (segment (start 170.925 111.25) (end 177.925 111.25) (width 0.25) (layer B.Cu) (net 19))
+  (segment (start 164.25 88.36) (end 166.88 85.73) (width 0.25) (layer B.Cu) (net 19))
+  (segment (start 164.25 109) (end 164.25 88.36) (width 0.25) (layer B.Cu) (net 19))
+  (segment (start 162.76 96.85) (end 166.88 100.97) (width 0.25) (layer F.Cu) (net 21))
+  (segment (start 160 96.85) (end 162.76 96.85) (width 0.25) (layer F.Cu) (net 21))
   (zone (net 1) (net_name GND) (layer F.Cu) (hatch edge 0.508)
     (connect_pads (clearance 0.508))

Commit message: cleanup resources and shield gerber files
Parts:
- removed JBTN0: Conn_01x03_Female, Connector_Wire:SolderWirePad_1x03_P3.175mm_Drill1mm
- added H2: MountingHole, MountingHole:MountingHole_2.2mm_M2, F.Cu at (188.5, 110.2)
- added JBUTTON0: Conn_01x02_Female, Connector_Wire:SolderWirePad_1x02_P3.81mm_Drill1mm, F.Cu at (160.0, 91.5)
- added R0: R_US, Resistor_THT:R_Axial_DIN0207_L6.3mm_D2.5mm_P7.62mm_Horizontal, F.Cu at (160.2, 107.0)
Routing:
- net Net-(JBUTTON0-Pad2): track 8.59 -> 18.4 mm
Other:
- board text added: "10K"
Changed lines of the file:
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@@
     (thickness 1.6)
     (drawings 51)
-    (tracks 28)
+    (tracks 31)
     (zones 0)
-    (modules 12)
+    (modules 14)
     (nets 23)
   )
@@
   (net 19 "Net-(JRGB0-Pad2)")
   (net 20 "Net-(U0-Pad13)")
-  (net 21 "Net-(JBTN0-Pad3)")
-  (net 22 "Net-(U0-Pad8)")
+  (net 21 "Net-(U0-Pad8)")
+  (net 22 "Net-(JBUTTON0-Pad2)")
   (net_class Default "This is the default net class."
     (clearance 0.2)
@@
     (uvia_drill 0.1)
     (add_net GND)
-    (add_net "Net-(JBTN0-Pad3)")
+    (add_net "Net-(JBUTTON0-Pad2)")
     (add_net "Net-(JEX0-Pad3)")
     (add_net "Net-(JRGB0-Pad2)")
@@
     (add_net VCC)
   )
+  (module Resistor_THT:R_Axial_DIN0207_L6.3mm_D2.5mm_P7.62mm_Horizontal (layer F.Cu)
+    (at 160.25 107 270)
+    (descr "Resistor, Axial_DIN0207 series, Axial, Horizontal, pin pitch=7.62mm, 0.25W = 1/4W, length*diameter=6.3*2.5mm^2, http://cdn-reichelt.de/documents/datenblatt/B400/1_4W%23YAG.pdf")
+    (tags "Resistor Axial_DIN0207 series Axial Horizontal pin pitch 7.62mm 0.25W = 1/4W length 6.3mm diameter 2.5mm")
+    (fp_text reference R0 (at 3.81 -2.37 90) (layer F.SilkS) hide
+      (effects (font (size 1 1) (thickness 0.15)))
+    )
+    (fp_text value R_US (at 3.81 2.37 90) (layer F.Fab)
+      (effects (font (size 1 1) (thickness 0.15)))
+    )
+    (fp_text user %R (at 3.81 0 90) (layer F.Fab)
+      (effects (font (size 1 1) (thickness 0.15)))
+    )
+    (fp_line (start 8.67 -1.5) (end -1.05 -1.5) (layer F.CrtYd) (width 0.05))
+    (fp_line (start 8.67 1.5) (end 8.67 -1.5) (layer F.CrtYd) (width 0.05))
+    (fp_line (start -1.05 1.5) (end 8.67 1.5) (layer F.CrtYd) (width 0.05))
+    (fp_line (start -1.05 -1.5) (end -1.05 1.5) (layer F.CrtYd) (width 0.05))
+    (fp_line (start 7.08 1.37) (end 7.08 1.04) (layer F.SilkS) (width 0.12))
+    (fp_line (start 0.54 1.37) (end 7.08 1.37) (layer F.SilkS) (width 0.12))
+    (fp_line (start 0.54 1.04) (end 0.54 1.37) (layer F.SilkS) (width 0.12))
+    (fp_line (start 7.08 -1.37) (end 7.08 -1.04) (layer F.SilkS) (width 0.12))
+    (fp_line (start 0.54 -1.37) (end 7.08 -1.37) (layer F.SilkS) (width 0.12))
+    (fp_line (start 0.54 -1.04) (end 0.54 -1.37) (layer F.SilkS) (width 0.12))
+    (fp_line (start 7.62 0) (end 6.96 0) (layer F.Fab) (width 0.1))
+    (fp_line (start 0 0) (end 0.66 0) (layer F.Fab) (width 0.1))
+    (fp_line (start 6.96 -1.25) (end 0.66 -1.25) (layer F.Fab) (width 0.1))
+    (fp_line (start 6.96 1.25) (end 6.96 -1.25) (layer F.Fab) (width 0.1))
+    (fp_line (start 0.66 1.25) (end 6.96 1.25) (layer F.Fab) (width 0.1))
+    (fp_line (start 0.66 -1.25) (end 0.66 1.25) (layer F.Fab) (width 0.1))
+    (pad 2 thru_hole oval (at 7.62 0 270) (size 1.6 1.6) (drill 0.8) (layers *.Cu *.Mask)
+      (net 1 GND))
+    (pad 1 thru_hole circle (at 0 0 270) (size 1.6 1.6) (drill 0.8) (layers *.Cu *.Mask)
+      (net 22 "Net-(JBUTTON0-Pad2)"))
+    (model ${KISYS3DMOD}/Resistor_THT.3dshapes/R_Axial_DIN0207_L6.3mm_D2.5mm_P7.62mm_Horizontal.wrl
+      (at (xyz 0 0 0))
+      (scale (xyz 1 1 1))
+      (rotate (xyz 0 0 0))
+    )
+  )
+  (module Connector_Wire:SolderWirePad_1x02_P3.81mm_Drill1mm (layer F.Cu)
+    (at 160 91.5 270)
+    (descr "Wire solder connection")
+    (tags connector)
+    (attr virtual)
+    (fp_text reference JBUTTON0 (at 1.905 -3.81 90) (layer F.SilkS) hide
+      (effects (font (size 1 1) (thickness 0.15)))
+    )
+    (fp_text value Conn_01x02_Female (at 1.905 3.81 90) (layer F.Fab)
+      (effects (font (size 1 1) (thickness 0.15)))
+    )
+    (fp_line (start 5.56 1.75) (end -1.74 1.75) (layer F.CrtYd) (width 0.05))
+    (fp_line (start 5.56 1.75) (end 5.56 -1.75) (layer F.CrtYd) (width 0.05))
+    (fp_line (start -1.74 -1.75) (end -1.74 1.75) (layer F.CrtYd) (width 0.05))
+    (fp_line (start -1.74 -1.75) (end 5.56 -1.75) (layer F.CrtYd) (width 0.05))
+    (fp_text user %R (at 1.905 0 90) (layer F.Fab)
+      (effects (font (size 1 1) (thickness 0.15)))
+    )
+    (pad 2 thru_hole circle (at 3.81 0 270) (size 2.49936 2.49936) (drill 1.00076) (layers *.Cu *.Mask)
+      (net 22 "Net-(JBUTTON0-Pad2)"))
+    (pad 1 thru_hole rect (at 0 0 270) (size 2.49936 2.49936) (drill 1.00076) (layers *.Cu *.Mask)
+      (net 2 VCC))
+  )
+  (module MountingHole:MountingHole_2.2mm_M2 (layer F.Cu)
+    (at 188.5 110.25)
+    (descr "Mounting Hole 2.2mm, no annular, M2")
+    (tags "mounting hole 2.2mm no annular m2")
+    (attr virtual)
+    (fp_text reference H2 (at 0 -3.2) (layer F.SilkS) hide
+      (effects (font (size 1 1) (thickness 0.15)))
+    )
+    (fp_text value MountingHole (at 0 3.2) (layer F.Fab)
+      (effects (font (size 1 1) (thickness 0.15)))
+    )
+    (fp_circle (center 0 0) (end 2.45 0) (layer F.CrtYd) (width 0.05))
+    (fp_circle (center 0 0) (end 2.2 0) (layer Cmts.User) (width 0.15))
+    (fp_text user %R (at 0.3 0) (layer F.Fab)
+      (effects (font (size 1 1) (thickness 0.15)))
+    )
+    (pad 1 np_thru_hole circle (at 0 0) (size 2.2 2.2) (drill 2.2) (layers *.Cu *.Mask))
+  )
   (module Connector_Wire:SolderWirePad_1x03_P3.175mm_Drill1mm (layer F.Cu)
     (at 160 80 270)
@@
     (pad 3 thru_hole circle (at 6.35 0 270) (size 2.49936 2.49936) (drill 1.00076) (layers *.Cu *.Mask)
       (net 18 "Net-(JEX0-Pad3)"))
-    (pad 2 thru_hole circle (at 3.175 0 270) (size 2.49936 2.49936) (drill 1.00076) (layers *.Cu *.Mask)
-      (net 1 GND))
-    (pad 1 thru_hole rect (at 0 0 270) (size 2.49936 2.49936) (drill 1.00076) (layers *.Cu *.Mask)
-      (net 2 VCC))
-  )
-  (module Connector_Wire:SolderWirePad_1x03_P3.175mm_Drill1mm (layer F.Cu)
-    (at 160 90.5 270)
-    (descr "Wire solder connection")
-    (tags connector)
-    (attr virtual)
-    (fp_text reference JBTN0 (at 3.175 -3.81 90) (layer F.SilkS) hide
-      (effects (font (size 1 1) (thickness 0.15)))
-    )
-    (fp_text value Conn_01x03_Female (at 3.175 3.175 90) (layer F.Fab)
-      (effects (font (size 1 1) (thickness 0.15)))
-    )
-    (fp_line (start 8.1 1.75) (end -1.74 1.75) (layer F.CrtYd) (width 0.05))
-    (fp_line (start 8.1 1.75) (end 8.1 -1.75) (layer F.CrtYd) (width 0.05))
-    (fp_line (start -1.74 -1.75) (end -1.74 1.75) (layer F.CrtYd) (width 0.05))
-    (fp_line (start -1.74 -1.75) (end 8.1 -1.75) (layer F.CrtYd) (width 0.05))
-    (fp_text user %R (at 3.175 0 90) (layer F.Fab)
-      (effects (font (size 1 1) (thickness 0.15)))
-    )
-    (pad 3 thru_hole circle (at 6.35 0 270) (size 2.49936 2.49936) (drill 1.00076) (layers *.Cu *.Mask)
-      (net 21 "Net-(JBTN0-Pad3)"))
     (pad 2 thru_hole circle (at 3.175 0 270) (size 2.49936 2.49936) (drill 1.00076) (layers *.Cu *.Mask)
       (net 1 GND))
@@
       (net 6 "Net-(U0-Pad24)"))
     (pad 12 thru_hole circle (at 13.97 7.62 270) (size 1.7526 1.7526) (drill 1.0922) (layers *.Cu *.SilkS *.Mask)
-      (net 21 "Net-(JBTN0-Pad3)"))
+      (net 22 "Net-(JBUTTON0-Pad2)"))
     (pad 23 thru_hole circle (at -11.43 -7.62 270) (size 1.7526 1.7526) (drill 1.0922) (layers *.Cu *.SilkS *.Mask)
       (net 1 GND))
@@
       (net 3 "Net-(JS0-Pad3)"))
     (pad 8 thru_hole circle (at 3.81 7.62 270) (size 1.7526 1.7526) (drill 1.0922) (layers *.Cu *.SilkS *.Mask)
-      (net 22 "Net-(U0-Pad8)"))
+      (net 21 "Net-(U0-Pad8)"))
     (pad 7 thru_hole circle (at 1.27 7.62 270) (size 1.7526 1.7526) (drill 1.0922) (layers *.Cu *.SilkS *.Mask)
       (net 18 "Net-(JEX0-Pad3)"))
@@
       (net 1 GND))
   )
+  (gr_text 10K (at 160.25 110.5 270) (layer F.SilkS)
+    (effects (font (size 1 1) (thickness 0.15)))
+  )
+  (gr_text "START BUTTON" (at 163.5 93.5 270) (layer F.SilkS)
+    (effects (font (size 1 1) (thickness 0.15)))
+  )
   (gr_text GND (at 162 83.25 270) (layer F.SilkS)
     (effects (font (size 1 1) (thickness 0.15)))
@@
     (effects (font (size 1 1) (thickness 0.15)))
   )
-  (gr_text D9 (at 162 97 270) (layer F.SilkS)
-    (effects (font (size 1 1) (thickness 0.15)))
-  )
-  (gr_text GND (at 162 93.75 270) (layer F.SilkS)
-    (effects (font (size 1 1) (thickness 0.15)))
-  )
-  (gr_text VCC (at 162 90.5 270) (layer F.SilkS)
-    (effects (font (size 1 1) (thickness 0.15)))
-  )
-  (gr_text "START BUTTON" (at 163.5 93.5 270) (layer F.SilkS)
+  (gr_text D9 (at 162 95.25 270) (layer F.SilkS)
+    (effects (font (size 1 1) (thickness 0.15)))
+  )
+  (gr_text VCC (at 162 91.5 270) (layer F.SilkS)
     (effects (font (size 1 1) (thickness 0.15)))
   )
@@
   (segment (start 164.25 88.36) (end 166.88 85.73) (width 0.25) (layer B.Cu) (net 19))
   (segment (start 164.25 109) (end 164.25 88.36) (width 0.25) (layer B.Cu) (net 19))
-  (segment (start 162.76 96.85) (end 166.88 100.97) (width 0.25) (layer F.Cu) (net 21))
-  (segment (start 160 96.85) (end 162.76 96.85) (width 0.25) (layer F.Cu) (net 21))
+  (segment (start 165.66 100.97) (end 166.88 100.97) (width 0.25) (layer F.Cu) (net 22))
+  (segment (start 160.25 107) (end 163.75 103.5) (width 0.25) (layer F.Cu) (net 22))
+  (segment (start 163.75 103.5) (end 163.75 99.25) (width 0.25) (layer F.Cu) (net 22))
+  (segment (start 163.75 99.25) (end 165.66 100.97) (width 0.25) (layer F.Cu) (net 22))
+  (segment (start 160 95.31) (end 163.75 99.25) (width 0.25) (layer F.Cu) (net 22))
   (zone (net 1) (net_name GND) (layer F.Cu) (hatch edge 0.508)
     (connect_pads (clearance 0.508))
