File: resources/kicad/pro_micro_shield/pro_micro_shield.kicad_sch (KiCad schematic)
At the start: 9 parts, among them J1 Conn_01x06_Female, J2 Conn_01x06_Female, J3 Conn_01x06_Female, J4 Conn_01x09_Female, U1 ProMicro

Commit message: shield revision 3
Parts:
- removed J2, J3: Conn_01x06_Female, Connector_PinHeader_2.54mm:PinHeader_1x06_P2.54mm_Vertical, symbol Connector:Conn_01x06_Female
- added J2: Conn_01x12_Female, Connector_PinHeader_2.54mm:PinHeader_1x12_P2.54mm_Vertical, symbol Connector:Conn_01x12_Female
- renumbered J4 to J3
Connections:
- net C6: now also J2.4 (Pin_4)
- net D4: now also J2.1 (Pin_1)
- net GND: now also J2.10 (Pin_10), J2.3 (Pin_3), J2.6 (Pin_6), J2.7 (Pin_7)
- net STRIP0: now also J2.11 (Pin_11), J2.8 (Pin_8)
- net VCC: now also J2.12 (Pin_12), J2.2 (Pin_2), J2.5 (Pin_5), J2.9 (Pin_9)
